File: kiCAD/FreeDSP-G_MAIN/ADC_DAC.sch (KiCad schematic (older format))
At the start: 148 parts, among them IC1 PCM5102APWR, IC2 PCM5102APWR, IC3 PCM1808QPWR, IC4 PCM1808QPWR, J11 Header_2P, J16 Header_3P, Q1 AO3400A, Q14 2SK30A-GR, Q2 2SK208GR, Q3 2SD2704KT146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

Commit message: Add files via upload
Parts:
- added C138: 220uF/10V, Capacitor_THT:CP_Radial_D7.5mm_P2.50mm, symbol Device:CP1_Small
- added C139: 470uF/16V, Capacitor_THT:CP_Radial_D10.0mm_P2.50mm_P5.00mm, symbol Device:CP1_Small
- C14: value 1uF -> 10uF/16V; JLPCB# C2158134 -> (none)
- R18: value 2.2MEG -> 1MEG
- R19: value 6.8k -> 100R; JLPCB# C23212 -> (none)
- R20: value 2.2k -> 1k
- R57: value 100k -> 0R
- R58: value 100k -> OR
Connections:
- net +10V: now also C139.1
- net GNDA: now also C138.2, C139.2
- net at Q14.1 (S), Q2.1 (S), R20.2: now also J16.3 (Pin_3); no longer C14.1
- net at Q14.3 (D), Q2.2 (D), R18.1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: now also C14.1, C138.1; no longer J16.3 (Pin_3)
Other:
- note added: "Buffer-AMP\n(-6dB)"
- note removed: "TRIODERISER\nHEAD-AMP\n(+18dB)"
- moved on the sheet: C14, Q14
Changed lines of the file:
@@
 Sheet 2 5
 Title "FreeDSP-G Schematic Circuit Diagram"
-Date "2025-02-01"
-Rev "0.1"
+Date "2025-05-19"
+Rev "0.3"
 Comp "CyberPit 2025"
 Comment1 ""
@@
 $EndComp
 Text Notes 3225 1475 0    79   ~ 0
-TRIODERISER\nHEAD-AMP\n(+18dB)
+Buffer-AMP\n(-6dB)
 $Comp
 L Device:R R?
@@
 P 4100 2075
 F 0 "Q2" H 4300 2125 50  0000 L CNN
-F 1 "2SK208GR" H 4300 2050 50  0000 L CNN
+F 1 "2SK208GR" H 4300 1950 50  0000 L CNN
 F 2 "TO_SOT_Packages_SMD:SC-59" H 4300 2175 50  0001 C CNN
 F 3 "~" H 4100 2075 50  0001 C CNN
@@
 P 4200 2500
 F 0 "R20" V 4100 2550 50  0000 R CNN
-F 1 "2.2k" V 4200 2575 50  0000 R CNN
+F 1 "1k" V 4200 2575 50  0000 R CNN
 F 2 "Resistor_SMD:R_0603_1608Metric_Pad0.98x0.95mm_HandSolder" V 4130 2500 50  0001 C CNN
 F 3 "~" H 4200 2500 50  0001 C CNN
@@
 P 4200 1275
 F 0 "R19" V 4100 1325 50  0000 R CNN
-F 1 "6.8k" V 4200 1350 50  0000 R CNN
+F 1 " 100R" V 4200 1400 50  0000 R CNN
 F 2 "Resistor_SMD:R_0603_1608Metric_Pad0.98x0.95mm_HandSolder" V 4130 1275 50  0001 C CNN
 F 3 "~" H 4200 1275 50  0001 C CNN
-F 4 "C23212" H 4200 1275 50  0001 C CNN "JLPCB#"
+F 4 "" H 4200 1275 50  0001 C CNN "JLPCB#"
 	1    4200 1275
 	-1   0    0    1
@@
 AR Path="/677034A1/697A9D89" Ref="R18"  Part="1"
 F 0 "R18" V 4075 1725 50  0000 C CNN
-F 1 "2.2MEG" V 3975 1675 50  0000 C CNN
+F 1 "1MEG" V 3975 1675 50  0000 C CNN
 F 2 "Resistor_SMD:R_0603_1608Metric_Pad0.98x0.95mm_HandSolder" V 3830 1675 50  0001 C CNN
 F 3 "" H 3900 1675 50  0001 C CNN
@@
 	3900 1525 3900 1475
 Wire Wire Line
-	3900 1475 4200 1475
-Wire Wire Line
 	4200 1475 4200 1425
 Connection ~ 4200 1475
@@
 L LPFS-21:CP_Small C14
 U 1 1 698EB12A
-P 4025 2500
-F 0 "C14" V 3800 2525 50  0000 C CNN
-F 1 "1uF" V 3875 2525 50  0000 C CNN
-F 2 "Capacitor_Tantalum_SMD:CP_EIA-2012-12_Kemet-R" H 4025 2500 50  0001 C CNN
-F 3 "~" H 4025 2500 50  0001 C CNN
-F 4 "C2158134" H 4025 2500 50  0001 C CNN "JLPCB#"
-	1    4025 2500
+P 5100 1625
+F 0 "C14" V 5000 1625 50  0000 C CNN
+F 1 "10uF/16V" V 4925 1575 50  0000 C CNN
+F 2 "Capacitor_Tantalum_SMD:CP_EIA-2012-12_Kemet-R" H 5100 1625 50  0001 C CNN
+F 3 "~" H 5100 1625 50  0001 C CNN
+F 4 "" H 5100 1625 50  0001 C CNN "JLPCB#"
+	1    5100 1625
 	1    0    0    -1
 $EndComp
 Wire Wire Line
-	4025 2400 4025 2325
-Wire Wire Line
-	4025 2325 4200 2325
-Wire Wire Line
-	4025 2600 4025 2675
-Connection ~ 4025 2675
-Wire Wire Line
-	4025 2675 4200 2675
-Wire Wire Line
 	3200 2675 3200 2450
 Wire Wire Line
@@
 Connection ~ 3475 2675
 Wire Wire Line
-	3475 2675 4025 2675
-Wire Wire Line
 	4200 1100 4200 1125
 Text Notes 3425 2450 1    50   ~ 0
@@
 L power:+10V #PWR?
 U 1 1 6AD1DA7B
-P 12150 8425
+P 12150 8050
 AR Path="/6889E617/6AD1DA7B" Ref="#PWR?"  Part="1"
 AR Path="/677034A1/6AD1DA7B" Ref="#PWR067"  Part="1"
-F 0 "#PWR067" H 12150 8275 50  0001 C CNN
-F 1 "+10V" H 12150 8575 50  0000 C CNN
-F 2 "" H 12150 8425 50  0001 C CNN
-F 3 "" H 12150 8425 50  0001 C CNN
-	1    12150 8425
+F 0 "#PWR067" H 12150 7900 50  0001 C CNN
+F 1 "+10V" H 12150 8200 50  0000 C CNN
+F 2 "" H 12150 8050 50  0001 C CNN
+F 3 "" H 12150 8050 50  0001 C CNN
+	1    12150 8050
 	1    0    0    -1
 $EndComp
@@
 Wire Wire Line
 	12275 8425 12150 8425
-Connection ~ 12150 8425
 Wire Wire Line
 	12475 8425 12650 8425
@@
 	0    -1   -1   0
 $EndComp
-$Comp
-L Device:CP1_Small C76
-U 1 1 6B3FB15E
-P 12925 8800
-F 0 "C76" V 13050 8800 50  0000 C CNN
-F 1 "220uF/10V" V 12800 8800 50  0000 C CNN
-F 2 "Capacitor_THT:CP_Radial_D7.5mm_P2.50mm" H 12925 8800 50  0001 C CNN
-F 3 "~" H 12925 8800 50  0001 C CNN
-F 4 "Low ESR will better for headphones coupling" H 12925 8800 50  0001 C CNN "Description"
-F 5 "HAND" H 12925 8800 50  0001 C CNN "JLPCB#"
-	1    12925 8800
-	0    -1   -1   0
-$EndComp
 Wire Wire Line
 	13000 7500 13175 7500
@@
 P 11525 7600
 F 0 "R58" V 11425 7550 50  0000 L CNN
-F 1 "100k" V 11525 7500 50  0000 L CNN
+F 1 "OR" V 11525 7550 50  0000 L CNN
 F 2 "Resistor_SMD:R_0603_1608Metric_Pad0.98x0.95mm_HandSolder" V 11455 7600 50  0001 C CNN
 F 3 "~" H 11525 7600 50  0001 C CNN
@@
 P 11500 8900
 F 0 "R57" V 11400 8850 50  0000 L CNN
-F 1 "100k" V 11500 8800 50  0000 L CNN
+F 1 "0R" V 11500 8850 50  0000 L CNN
 F 2 "Resistor_SMD:R_0603_1608Metric_Pad0.98x0.95mm_HandSolder" V 11430 8900 50  0001 C CNN
 F 3 "~" H 11500 8900 50  0001 C CNN
@@
 Wire Notes Line
 	3600 3000 3475 3000
-Text Notes 1350 3050 0    50   ~ 0
+Text Notes 1250 3050 0    50   ~ 0
 Change to 1uF for pre-emphasis normalized overdrive.\n(De-emphasis shoud have done in DSP processing)
 Wire Wire Line
@@
 Wire Wire Line
 	3650 5600 2500 5600
-Wire Wire Line
-	4200 2325 5100 2325
 $Comp
 L Device:Q_NJFET_SGD Q14
 U 1 1 67C8CC1F
-P 5000 2075
-F 0 "Q14" H 5200 2125 50  0000 L CNN
-F 1 "2SK30A-GR" H 5200 2050 50  0000 L CNN
-F 2 "TO_SOT_Packages_THT:TO-92_Inline_Narrow_Oval" H 5200 2175 50  0001 C CNN
-F 3 "~" H 5000 2075 50  0001 C CNN
-F 4 "Replace of 2SK30A" H 5000 2075 50  0001 C CNN "Description"
-F 5 "C2999170" H 5000 2075 50  0001 C CNN "JLPCB#"
-	1    5000 2075
+P 4750 2075
+F 0 "Q14" H 4950 2125 50  0000 L CNN
+F 1 "2SK30A-GR" H 4950 2050 50  0000 L CNN
+F 2 "TO_SOT_Packages_THT:TO-92_Inline_Narrow_Oval" H 4950 2175 50  0001 C CNN
+F 3 "~" H 4750 2075 50  0001 C CNN
+F 4 "Replace of 2SK30A" H 4750 2075 50  0001 C CNN "Description"
+F 5 "C2999170" H 4750 2075 50  0001 C CNN "JLPCB#"
+	1    4750 2075
 	1    0    0    -1
 $EndComp
 Wire Wire Line
-	5100 2275 5100 2325
-Wire Wire Line
-	4200 1475 5100 1475
+	4850 2275 4850 2325
 Wire Wire Line
 	3900 1825 3900 1850
@@
 	4200 1475 4200 1875
 Wire Wire Line
-	3900 1850 4775 1850
-Wire Wire Line
-	4775 1850 4775 2075
+	4525 1850 4525 2075
 Wire Wire Line
-	4775 2075 4800 2075
+	4525 2075 4550 2075
 Connection ~ 3900 1850
 Wire Wire Line
 	3900 1850 3900 2075
 Wire Notes Line
-	4450 2175 5200 3025
+	4525 2275 5175 3000
 Wire Notes Line
-	5200 3025 5400 2200
+	5200 3025 5075 2175
 Text Notes 4700 3200 0    50   ~ 0
 ALTERNATIVE CHOICE\nSELECT ONE AS YOU LIKE
@@
 	5600 975  5600 800
 Wire Wire Line
-	5600 1175 5600 1475
+	5600 1175 5600 2325
 Wire Wire Line
-	5600 1475 5100 1475
+	5600 2325 4850 2325
 Wire Wire Line
 	5525 1175 5600 1175
@@
 Wire Notes Line width 16 style solid
 	5175 1100 5175 1200
-Connection ~ 5100 1475
 Wire Wire Line
-	5100 1475 5100 1875
+	4850 1475 4850 1875
 Text Notes 6375 3075 0    50   ~ 0
 ※
@@
 Text Notes 8450 2225 0    50   ~ 0
 1.42V
+Connection ~ 4850 2325
+Wire Wire Line
+	4200 2325 4850 2325
+Wire Wire Line
+	4200 1475 4850 1475
+Wire Wire Line
+	3900 1850 4525 1850
+Wire Wire Line
+	3900 1475 4200 1475
+Wire Wire Line
+	3475 2675 4200 2675
+$Comp
+L power:GNDA #PWR?
+U 1 1 686841EF
+P 5100 1750
+AR Path="/686841EF" Ref="#PWR?"  Part="1"
+AR Path="/5D67FDC6/686841EF" Ref="#PWR?"  Part="1"
+AR Path="/5D902CF8/686841EF" Ref="#PWR?"  Part="1"
+AR Path="/6787F48A/5D902CF8/686841EF" Ref="#PWR?"  Part="1"
+AR Path="/67A62685/686841EF" Ref="#PWR?"  Part="1"
+AR Path="/677034A1/686841EF" Ref="#PWR0148"  Part="1"
+F 0 "#PWR0148" H 5100 1500 50  0001 C CNN
+F 1 "GNDA" H 5100 1600 50  0000 C CNN
+F 2 "" H 5100 1750 50  0001 C CNN
+F 3 "" H 5100 1750 50  0001 C CNN
+	1    5100 1750
+	1    0    0    -1
+$EndComp
+Wire Wire Line
+	5100 1725 5100 1750
+Wire Wire Line
+	5100 1525 5100 1475
+Wire Wire Line
+	5100 1475 4850 1475
+Connection ~ 4850 1475
+$Comp
+L Device:CP1_Small C138
+U 1 1 68406942
+P 5275 1625
+F 0 "C138" V 5375 1625 50  0000 C CNN
+F 1 "220uF/10V" V 5450 1600 50  0000 C CNN
+F 2 "Capacitor_THT:CP_Radial_D7.5mm_P2.50mm" H 5275 1625 50  0001 C CNN
+F 3 "~" H 5275 1625 50  0001 C CNN
+F 4 "Low ESR will better for headphones coupling" H 5275 1625 50  0001 C CNN "Description"
+F 5 "HAND" H 5275 1625 50  0001 C CNN "JLPCB#"
+	1    5275 1625
+	1    0    0    -1
+$EndComp
+Wire Wire Line
+	5275 1525 5275 1475
+Wire Wire Line
+	5275 1475 5100 1475
+Connection ~ 5100 1475
+Wire Wire Line
+	5275 1750 5100 1750
+Wire Wire Line
+	5275 1725 5275 1750
+Connection ~ 5100 1750
+$Comp
+L Device:CP1_Small C76
+U 1 1 6B3FB15E
+P 12925 8800
+F 0 "C76" V 13050 8800 50  0000 C CNN
+F 1 "220uF/10V" V 12800 8800 50  0000 C CNN
+F 2 "Capacitor_THT:CP_Radial_D7.5mm_P2.50mm" H 12925 8800 50  0001 C CNN
+F 3 "~" H 12925 8800 50  0001 C CNN
+F 4 "Low ESR will better for headphones coupling" H 12925 8800 50  0001 C CNN "Description"
+F 5 "HAND" H 12925 8800 50  0001 C CNN "JLPCB#"
+	1    12925 8800
+	0    -1   -1   0
+$EndComp
+Wire Wire Line
+	12150 8050 12150 8425
+Connection ~ 12150 8425
+$Comp
+L Device:CP1_Small C139
+U 1 1 68AA8EEE
+P 11550 8300
+F 0 "C139" V 11675 8300 50  0000 C CNN
+F 1 "470uF/16V" V 11425 8300 50  0000 C CNN
+F 2 "Capacitor_THT:CP_Radial_D10.0mm_P2.50mm_P5.00mm" H 11550 8300 50  0001 C CNN
+F 3 "~" H 11550 8300 50  0001 C CNN
+F 4 "Low ESR will better for headphones coupling" H 11550 8300 50  0001 C CNN "Description"
+F 5 "HAND" H 11550 8300 50  0001 C CNN "JLPCB#"
+	1    11550 8300
+	1    0    0    -1
+$EndComp
+$Comp
+L power:+10V #PWR?
+U 1 1 68AA8EF4
+P 11550 8150
+AR Path="/6889E617/68AA8EF4" Ref="#PWR?"  Part="1"
+AR Path="/677034A1/68AA8EF4" Ref="#PWR0149"  Part="1"
+F 0 "#PWR0149" H 11550 8000 50  0001 C CNN
+F 1 "+10V" H 11550 8325 50  0000 C CNN
+F 2 "" H 11550 8150 50  0001 C CNN
+F 3 "" H 11550 8150 50  0001 C CNN
+	1    11550 8150
+	1    0    0    -1
+$EndComp
+Wire Wire Line
+	11550 8150 11550 8200
+Wire Wire Line
+	11550 8400 11550 8450
+$Comp
+L power:GNDA #PWR?
+U 1 1 68BAC56B
+P 11550 8450
+AR Path="/68BAC56B" Ref="#PWR?"  Part="1"
+AR Path="/5D67FDC6/68BAC56B" Ref="#PWR?"  Part="1"
+AR Path="/5D902CF8/68BAC56B" Ref="#PWR?"  Part="1"
+AR Path="/6787F48A/5D902CF8/68BAC56B" Ref="#PWR?"  Part="1"
+AR Path="/67A62685/68BAC56B" Ref="#PWR?"  Part="1"
+AR Path="/677034A1/68BAC56B" Ref="#PWR0150"  Part="1"
+F 0 "#PWR0150" H 11550 8200 50  0001 C CNN
+F 1 "GNDA" H 11550 8300 50  0000 C CNN
+F 2 "" H 11550 8450 50  0001 C CNN
+F 3 "" H 11550 8450 50  0001 C CNN
+	1    11550 8450
+	1    0    0    -1
+$EndComp
 $EndSCHEMATC
