File: kiCAD/FreeDSP-G_MAIN/BM83_BT-RX.sch (KiCad schematic (older format))
At the start: 16 parts, among them J17 5077CR-16-SMC2, J18 Header_2P, J19 Header_6P, SW2 TVBP06, U14 BM83

Commit message: Add files via upload
Parts:
- added D14, D9: B5819W SL, Diode_SMD:D_SOD-123, symbol Diode:BAT43W-V
- added FB18: GZ1608D601TF, Inductor_SMD:L_0603_1608Metric_Pad1.05x0.95mm_HandSolder, symbol ferrite_bead:Ferrite_Bead
- added SW3: MFB, Button_Switch_THT:SW_Tactile_SPST_Angled_PTS645Vx83-2LFS, symbol dk_Pushbutton-Switches:GPTS203211B
Connections:
- net VBUS: now also D14.1 (K), D9.1 (K); no longer J17.A4 (VBUS), J17.A9 (VBUS), J17.B4 (VBUS), J17.B9 (VBUS)
- net at C131.1, D12.2 (A), D13.2 (A)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: now also SW3.1
- net at C131.2, SW2.1, U14.26 (PWRMFB): now also SW3.2
- new net: D14.2 (A), J17.A4 (VBUS), J17.A9 (VBUS), J17.B4 (VBUS), J17.B9 (VBUS)
- new net: D9.2 (A), FB18.2
- new net +5VA: FB18.1
Changed lines of the file:
@@
 Sheet 5 5
 Title "FreeDSP-G Schematic Circuit Diagram"
-Date "2025-02-01"
-Rev "0.1"
+Date "2025-05-19"
+Rev "0.3"
 Comp "CyberPit 2025"
 Comment1 ""
@@
 AR Path="/6811C4A3/6812DEBA" Ref="FB17"  Part="1"
 F 0 "FB17" V 1300 4475 60  0000 C CNN
-F 1 "GZ1608D601TF" V 1200 4475 60  0000 C CNN
+F 1 "GZ1608D601TF" V 1225 4625 60  0000 C CNN
 F 2 "Inductor_SMD:L_0603_1608Metric_Pad1.05x0.95mm_HandSolder" H 1600 4675 60  0001 L CNN
 F 3 "https://www.murata.com/en-us/products/productdata/8796738650142/ENFA0003.pdf" H 1600 4775 60  0001 L CNN
@@
 Wire Wire Line
 	8725 4000 8825 4000
-Wire Wire Line
-	1525 4375 3400 4375
 Text Label 1525 4375 0    50   ~ 0
 VBUS
 Wire Wire Line
 	8225 1650 7525 1650
-Text Label 7100 1650 0    50   ~ 0
+Text Label 6500 1650 0    50   ~ 0
 VBUS
 Wire Wire Line
@@
 Connection ~ 7675 3350
 Connection ~ 8300 4000
-Text Notes 1100 5425 0    98   ~ 20
+Text Notes 800  5425 0    98   ~ 20
 Multi\nFunction\nButton
 Text Notes 7850 2275 0    50   ~ 0
@@
 Wire Wire Line
 	2575 2275 3400 2275
+$Comp
+L Diode:BAT43W-V D?
+U 1 1 68339A60
+P 6950 1650
+AR Path="/5D60B524/68339A60" Ref="D?"  Part="1"
+AR Path="/68339A60" Ref="D?"  Part="1"
+AR Path="/6787F48A/68339A60" Ref="D?"  Part="1"
+AR Path="/6889E617/68339A60" Ref="D?"  Part="1"
+AR Path="/6811C4A3/68339A60" Ref="D14"  Part="1"
+F 0 "D14" H 6950 1775 50  0000 C CNN
+F 1 "B5819W SL" H 6925 1550 50  0000 C CNN
+F 2 "Diode_SMD:D_SOD-123" H 6950 1475 50  0001 C CNN
+F 3 "http://www.vishay.com/docs/85660/bat42.pdf" H 6950 1650 50  0001 C CNN
+F 4 "C8598" H 6950 1650 50  0001 C CNN "JLPCB#"
+F 5 "SBD 1A/40V" H 6950 1650 50  0001 C CNN "Description"
+	1    6950 1650
+	1    0    0    -1
+$EndComp
+Wire Wire Line
+	6500 1650 6800 1650
+$Comp
+L Diode:BAT43W-V D?
+U 1 1 683407FE
+P 1350 4075
+AR Path="/5D60B524/683407FE" Ref="D?"  Part="1"
+AR Path="/683407FE" Ref="D?"  Part="1"
+AR Path="/6787F48A/683407FE" Ref="D?"  Part="1"
+AR Path="/6889E617/683407FE" Ref="D?"  Part="1"
+AR Path="/6811C4A3/683407FE" Ref="D9"  Part="1"
+F 0 "D9" H 1350 4200 50  0000 C CNN
+F 1 "B5819W SL" H 1325 3975 50  0000 C CNN
+F 2 "Diode_SMD:D_SOD-123" H 1350 3900 50  0001 C CNN
+F 3 "http://www.vishay.com/docs/85660/bat42.pdf" H 1350 4075 50  0001 C CNN
+F 4 "C8598" H 1350 4075 50  0001 C CNN "JLPCB#"
+F 5 "SBD 1A/40V" H 1350 4075 50  0001 C CNN "Description"
+	1    1350 4075
+	0    -1   -1   0
+$EndComp
+Wire Wire Line
+	1350 4225 1350 4375
+Wire Wire Line
+	1350 4375 3400 4375
+$Comp
+L power:+5VA #PWR?
+U 1 1 68349098
+P 1350 3525
+AR Path="/67A62685/68349098" Ref="#PWR?"  Part="1"
+AR Path="/6787F48A/68349098" Ref="#PWR?"  Part="1"
+AR Path="/6889E617/68349098" Ref="#PWR?"  Part="1"
+AR Path="/6811C4A3/68349098" Ref="#PWR0147"  Part="1"
+F 0 "#PWR0147" H 1350 3375 50  0001 C CNN
+F 1 "+5VA" H 1350 3675 50  0000 C CNN
+F 2 "" H 1350 3525 50  0001 C CNN
+F 3 "" H 1350 3525 50  0001 C CNN
+	1    1350 3525
+	1    0    0    -1
+$EndComp
+$Comp
+L ferrite_bead:Ferrite_Bead FB?
+U 1 1 6834BA5A
+P 1350 3725
+AR Path="/677034A1/6834BA5A" Ref="FB?"  Part="1"
+AR Path="/6823265E/6834BA5A" Ref="FB?"  Part="1"
+AR Path="/6811C4A3/6834BA5A" Ref="FB18"  Part="1"
+F 0 "FB18" V 1250 3725 60  0000 C CNN
+F 1 "GZ1608D601TF" V 1150 3725 60  0000 C CNN
+F 2 "Inductor_SMD:L_0603_1608Metric_Pad1.05x0.95mm_HandSolder" H 1550 3925 60  0001 L CNN
+F 3 "https://www.murata.com/en-us/products/productdata/8796738650142/ENFA0003.pdf" H 1550 4025 60  0001 L CNN
+F 4 "490-1014-1-ND" H 1550 4125 60  0001 L CNN "Digi-Key_PN"
+F 5 "BLM18AG601SN1D" H 1550 4225 60  0001 L CNN "MPN"
+F 6 "Filters" H 1550 4325 60  0001 L CNN "Category"
+F 7 "Ferrite Beads and Chips" H 1550 4425 60  0001 L CNN "Family"
+F 8 "https://www.murata.com/en-us/products/productdata/8796738650142/ENFA0003.pdf" H 1550 4525 60  0001 L CNN "DK_Datasheet_Link"
+F 9 "/product-detail/en/murata-electronics-north-america/BLM18AG601SN1D/490-1014-1-ND/584462" H 1550 4625 60  0001 L CNN "DK_Detail_Page"
+F 10 "FERRITE BEAD 600 OHM 0603 1LN" H 1550 4725 60  0001 L CNN "Description"
+F 11 "Murata Electronics North America" H 1550 4825 60  0001 L CNN "Manufacturer"
+F 12 "Active" H 1550 4925 60  0001 L CNN "Status"
+F 13 "C1002" H 1350 3725 50  0001 C CNN "JLPCB#"
+	1    1350 3725
+	1    0    0    -1
+$EndComp
+Wire Wire Line
+	1350 3525 1350 3575
+Wire Wire Line
+	1350 3875 1350 3925
+$Comp
+L dk_Pushbutton-Switches:GPTS203211B SW?
+U 1 1 68317849
+P 1625 5225
+AR Path="/68317849" Ref="SW?"  Part="1"
+AR Path="/5D902CF8/68317849" Ref="SW?"  Part="1"
+AR Path="/6787F48A/5D902CF8/68317849" Ref="SW?"  Part="1"
+AR Path="/67A62685/68317849" Ref="SW?"  Part="1"
+AR Path="/677034A1/68317849" Ref="SW?"  Part="1"
+AR Path="/6823265E/68317849" Ref="SW?"  Part="1"
+AR Path="/6811C4A3/68317849" Ref="SW3"  Part="1"
+F 0 "SW3" V 1650 5200 50  0000 R CNN
+F 1 "MFB" V 1575 5200 50  0000 R CNN
+F 2 "Button_Switch_THT:SW_Tactile_SPST_Angled_PTS645Vx83-2LFS" H 1625 5425 50  0001 C CNN
+F 3 "" H 1625 5425 50  0001 C CNN
+F 4 "HAND" H 1625 5225 50  0001 C CNN "JLPCB#"
+F 5 "for manual reset button for DSP" H 1625 5225 50  0001 C CNN "Description"
+	1    1625 5225
+	0    -1   1    0
+$EndComp
+Wire Wire Line
+	1625 5425 1625 5550
+Wire Wire Line
+	1625 5550 1950 5550
+Connection ~ 1950 5550
+Wire Wire Line
+	1625 5025 1625 4575
+Wire Wire Line
+	1625 4575 1950 4575
+Connection ~ 1950 4575
 $EndSCHEMATC
