File: kiCAD/FreeDSP-G_MAIN/DSP.sch (KiCad schematic (older format))
At the start: 89 parts, among them J12 Conn_01x08, J13 IDC_2x5, J14 Conn_01x08, J15 Conn_01x08, Q10 B772M, Q11 AO3401A, Q12 AO3400A, Q13 AO3400A, SW1 DSP_RES, U11 74LVC1G04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

Commit message: Add files via upload
Parts:
- added D15: B5819W SL, Diode_SMD:D_SOD-123, symbol Diode:BAT43W-V
- added R130, R131, R132: NOP, Resistor_SMD:R_0603_1608Metric_Pad0.98x0.95mm_HandSolder, symbol Device:R
- added R82: 100k, Resistor_SMD:R_0603_1608Metric_Pad0.98x0.95mm_HandSolder, symbol Device:R
Connections:
- net +3V3: now also R82.1
- net BCK_IN2: now also R132.1
- net BCK_OUT2: now also R132.2
- net BT_TXD: now also R130.1
- net DAT_OUT2: now also R130.2
- net LRK_IN2: now also R131.1
- net LRK_OUT2: now also R131.2
- net ~DSP-RESET: now also D15.2 (A); no longer C137.1
- new net: C137.1, D15.1 (K), R82.2
Other:
- moved on the sheet: C130, FB14, J12, J14, J15, R114
