File: kiCAD/FreeDSP-G_MAIN/FreeDSP-G.kicad_pcb (KiCad board)
At the start: 4 copper layers, 170 x 101 mm, 366 parts, among them IC1 PCM5102APWR, IC2 PCM5102APWR, IC3 PCM1808QPWR, IC4 PCM1808QPWR, IC5 TPS5430DDA, J1 NMJ6HCD2, J10 NMJ6HCD2, J11 Header_2P, J12 Conn_01x08, J13 IDC_2x5, J14 Conn_01x08, J15 Conn_01x08, J16 Header_3P, J17 5077CR-16-SMC2, J18 Header_2P, J19 Header_6P, J2 NMJ6HCD2, J3 TRS-mini, J4 Barrel_Jack_Switch, J5 Conn_02x07_Odd_Even, J6 Conn_02x05_Odd_Even, J7 NMJ6HCD2, J8 SJ1-3535NG, J9 NMJ6HCD2, Q1 AO3400A, Q10 B772M, Q11 AO3401A, Q12 AO3400A, Q13 AO3400A, Q14 2SK30A-GR, Q2 2SK208GR, Q3 2SD2704KT146, Q4 2SD2704KT146, Q5 MMBT5401, Q6 MMBT5401, Q8 AO3401A, Q9 AO3400A, SW1 DSP_RES, SW2 TVBP06, U1 PLR135-T10, U10 LM317AG-TN3-R, U11 74LVC1G04, U12 ADAU1467, U13 25AA1024(512), U14 BM83, U2 PLT133-T10W, U3 XIAO_RP2040, U4 OPA1678IDR, U5 OPA1678IDR, U6 OPA1678IDR, U7 NJM4556AD, U8 LM317AG-TN3-R, U9 AMS1117-3.3, Y1 OT322512.288MJBA4S

Commit message: Add files via upload
Parts:
- added C138: 220uF/10V, Capacitor_THT:CP_Radial_D7.5mm_P2.50mm, F.Cu at (215.7, 89.8)
- added C139: 470uF/16V, Capacitor_THT:CP_Radial_D10.0mm_P2.50mm_P5.00mm, F.Cu at (208.1, 95.8)
- added D14: B5819W SL, Diode_SMD:D_SOD-123, F.Cu at (195.0, 130.2)
- added D15: B5819W SL, Diode_SMD:D_SOD-123, F.Cu at (181.3, 134.6)
- added D9: B5819W SL, Diode_SMD:D_SOD-123, F.Cu at (194.6, 122.6)
- added FB18: GZ1608D601TF, Inductor_SMD:L_0603_1608Metric_Pad1.05x0.95mm_HandSolder, F.Cu at (184.4, 123.5)
- added R130: NOP, Resistor_SMD:R_0603_1608Metric_Pad0.98x0.95mm_HandSolder, F.Cu at (193.1, 109.7)
- added R131: NOP, Resistor_SMD:R_0603_1608Metric_Pad0.98x0.95mm_HandSolder, F.Cu at (193.1, 116.8)
- added R132: NOP, Resistor_SMD:R_0603_1608Metric_Pad0.98x0.95mm_HandSolder, F.Cu at (193.1, 113.2)
- added R82: 100k, Resistor_SMD:R_0603_1608Metric_Pad0.98x0.95mm_HandSolder, F.Cu at (179.7, 131.2)
- added SW3: MFB, Button_Switch_THT:SW_Tactile_SPST_Angled_PTS645Vx83-2LFS, F.Cu at (217.2, 106.9)
- C14: value 1uF -> 10uF/16V
- R18: value 2.2MEG -> 1MEG
- R19: value 6.8k -> 100R
- R20: value 2.2k -> 1k
- R57: value 100k -> 0R
- R58: value 100k -> OR
- SW2: moved to B.Cu
- moved D12 47.5 mm to (218.5, 102.3)
- moved D13 38.2 mm to (218.4, 116.2), turned to 90 degrees
- moved C137 36.8 mm to (181.2, 128.3), turned to 90 degrees
- moved SW2 8.28 mm to (208.2, 112.5)
- moved C11 6.97 mm to (210.8, 69.2)
- moved R14 4.03 mm to (201.8, 67.7), turned to 0 degrees
- moved C13 3.93 mm to (204.3, 69.9), turned to 0 degrees
- moved C131 3.05 mm to (191.6, 131.7), turned to 0 degrees
- moved R12 0.69 mm to (204.5, 66.8), turned to 270 degrees
- moved R18 0.21 mm to (199.6, 74.4)
Connections:
- C137 pad 1: ~DSP-RESET -> Net-(C137-Pad1)
- C14 pad 1: Net-(C14-Pad1) -> Net-(C138-Pad1)
- J17 pad A4: /BM83_BT-RX/VBUS -> Net-(D14-Pad2)
- J17 pad A9: /BM83_BT-RX/VBUS -> Net-(D14-Pad2)
- J17 pad B4: /BM83_BT-RX/VBUS -> Net-(D14-Pad2)
- J17 pad B9: /BM83_BT-RX/VBUS -> Net-(D14-Pad2)
- Q14 pad 1: Net-(C14-Pad1) -> Net-(J16-Pad3)
- Q14 pad 3: Net-(J16-Pad3) -> Net-(C138-Pad1)
- Q2 pad 1: Net-(C14-Pad1) -> Net-(J16-Pad3)
- Q2 pad 2: Net-(J16-Pad3) -> Net-(C138-Pad1)
- R18 pad 1: Net-(J16-Pad3) -> Net-(C138-Pad1)
- R19 pad 1: Net-(J16-Pad3) -> Net-(C138-Pad1)
- R20 pad 2: Net-(C14-Pad1) -> Net-(J16-Pad3)
Routing:
- net Net-(D12-Pad1): track 11.9 -> 46.0 mm, vias 0 -> 2
- net Net-(C138-Pad1): track 0.00 -> 30.9 mm
- net Net-(D14-Pad2): track 0.00 -> 23.2 mm, vias 0 -> 3
- net /BM83_BT-RX/VBUS: track 27.8 -> 9.26 mm, vias 3 -> 0
- net Net-(D13-Pad1): track 12.6 -> 31.1 mm, vias 0 -> 2
- net Net-(C131-Pad2): track 35.9 -> 50.1 mm
- net Net-(C14-Pad1): track 14.2 -> 0.00 mm
- net Net-(D9-Pad2): track 0.00 -> 8.56 mm
- net Net-(C131-Pad1): track 62.8 -> 71.1 mm, vias 3 -> 1
- net Net-(C11-Pad2): track 9.93 -> 2.97 mm
- net GND: track 415.7 -> 422.4 mm
- net DAT_OUT2: track 32.1 -> 37.2 mm
- net BCK_OUT2: track 36.6 -> 41.3 mm
- net EX_SDA: track 154.9 -> 150.3 mm
- net +3V3: track 294.4 -> 298.8 mm
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Other:
- board text added: "Multi Function BUTTON"
- board text added: "Version 0.3"
- board text removed: "Version 0.2"
