File: kiCAD/FreeDSP-G_MAIN/FreeDSP-G.sch (KiCad schematic (older format))
At the start: 44 parts, among them J1 NMJ6HCD2, J10 NMJ6HCD2, J2 NMJ6HCD2, J3 TRS-mini, J4 Barrel_Jack_Switch, J5 Conn_02x07_Odd_Even, J6 Conn_02x05_Odd_Even, J7 NMJ6HCD2, J8 SJ1-3535NG, J9 NMJ6HCD2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

Commit message: Add files via upload
Changed lines of the file:
@@
 Sheet 1 5
 Title "FreeDSP-G Schematic Circuit Diagram"
-Date "2025-02-20"
-Rev "0.2"
+Date "2025-05-19"
+Rev "0.3"
 Comp "CyberPit 2025"
 Comment1 "(Without BM83 version)"
@@
 	2325 1100 8100 1075
 $Sheet
-S 6525 9200 4625 1575
+S 6525 9225 4625 1575
 U 6889E617
 F0 "PSU" 118
