File: kiCAD/FreeDSP-G_MAIN/PSU.sch (KiCad schematic (older format))
At the start: 66 parts, among them IC5 TPS5430DDA, Q5 MMBT5401, Q6 MMBT5401, Q8 AO3401A, Q9 AO3400A, U10 LM317AG-TN3-R, U8 LM317AG-TN3-R, U9 AMS1117-3.3

Commit message: Add files via upload
Changed lines of the file:
@@
 Sheet 3 5
 Title "FreeDSP-G Schematic Circuit Diagram"
-Date "2025-02-27"
-Rev "0.2"
+Date "2025-05-19"
+Rev "0.3"
 Comp "CyberPit 2025"
 Comment1 ""
@@
 	1    0    0    -1
 $EndComp
-Text Notes 4000 3725 0    50   ~ 0
+Text Notes 3900 3750 0    50   ~ 0
 (ADC/DAC/Line-Driver Power)
 $Comp
